File: Electronica Kicad/Cs Naturales.kicad_pcb (KiCad board)
At the start: 2 copper layers, 7 parts

Commit message: Diseño PCB listo
Parts:
- removed U2: ~, Librerias:ESP32-DevKit_V1
- added ?: , , F.Cu at (89.6, 74.6)
- added ?: , , F.Cu at (89.6, 69.1)
- added ?: , , F.Cu at (89.6, 72.1)
- added H4: Sujeción, MountingHole:MountingHole_3.5mm_Pad, F.Cu at (66.0, 134.0)
- added H4: Sujeción, MountingHole:MountingHole_3.5mm_Pad, F.Cu at (137.0, 62.5)
- added H4: Sujeción, MountingHole:MountingHole_3.5mm_Pad, F.Cu at (65.5, 62.0)
- added H4: Sujeción, MountingHole:MountingHole_3.5mm_Pad, F.Cu at (137.0, 134.0)
- added REF**: C_Disc_D7.5mm_W4.4mm_P5.00mm, Capacitor_THT:C_Disc_D7.5mm_W4.4mm_P5.00mm, F.Cu at (120.0, 89.0)
- added REF**: C_Disc_D7.5mm_W4.4mm_P5.00mm, Capacitor_THT:C_Disc_D7.5mm_W4.4mm_P5.00mm, F.Cu at (120.5, 109.8)
- added REF**: C_Disc_D7.5mm_W4.4mm_P5.00mm, Capacitor_THT:C_Disc_D7.5mm_W4.4mm_P5.00mm, F.Cu at (73.0, 82.5)
- added S1: Conn_01x04_MountingPin, Connector_PinHeader_2.54mm:PinHeader_1x04_P2.54mm_Vertical, F.Cu at (79.5, 88.0)
- added S2: Conn_01x05_MountingPin, Connector_PinHeader_2.54mm:PinHeader_1x05_P2.54mm_Vertical, F.Cu at (125.0, 83.5)
- added S3: Conn_01x06_MountingPin, Connector_PinHeader_2.54mm:PinHeader_1x06_P2.54mm_Vertical, F.Cu at (125.0, 93.5)
- M1: footprint Librerias1:ESP32-DevKit_V1 -> ESP32_ Naturales:ESP32-DevKit_V1
- moved R1 57.5 mm to (88.5, 68.0)
- moved D1 50.3 mm to (108.2, 63.0), turned to 0 degrees
- moved R2 46.4 mm to (116.0, 68.5), turned to 180 degrees
- moved D2 40.3 mm to (96.0, 63.0), turned to 180 degrees
- moved B1 5.13 mm to (98.4, 130.5), turned to 0 degrees
- moved M1 0.62 mm to (89.1, 77.2)
Connections:
- B1 pad 1: GND_IN -> GND_In
- B1 pad 2: VIN -> Vin
- M1 pad 10: LED_WIFI -> LED_ON
- M1 pad 11: unconnected-(M1-D14/ADC2_6/HSPI_CLK/T6/~-Pad11) -> D14
- M1 pad 13: unconnected-(M1-D13/ADC2_4/HSPI_ID/T4/~-Pad13) -> D13
- M1 pad 14: VIN -> GND_In
- M1 pad 15: GND_IN -> Vin
- M1 pad 4: S1 A0 -> S1 D0
- M1 pad 5: unconnected-(M1-D35/ADC1_7-Pad5) -> D35
- M1 pad 6: unconnected-(M1-D32/ADC1_2/~-Pad6) -> D32
- M1 pad 7: unconnected-(M1-D33/ADC1_5/T8/~-Pad7) -> D33
- M1 pad 8: S1 D0 -> S1 A0
- M1 pad 9: LED_ON -> LED_WIFI
Routing:
- net GND: track 0.00 -> 299.6 mm
- net S1 +: track 0.00 -> 297.8 mm, vias 0 -> 2
- net LED_ON: track 0.00 -> 60.0 mm, vias 0 -> 2
- net S2 SDA: track 0.00 -> 49.9 mm, vias 0 -> 2
- net S2 SCL: track 0.00 -> 42.6 mm
- net LED_WIFI: track 0.00 -> 40.3 mm
- net VIN: track 33.8 -> 0.00 mm
- net GND_In: track 0.00 -> 33.8 mm
- net GND_IN: track 30.7 -> 0.00 mm
- net Vin: track 0.00 -> 29.6 mm
- net S1 D0: track 0.00 -> 16.0 mm
- net S1 A0: track 0.00 -> 10.6 mm
- net Net-(D1-A): track 0.00 -> 5.58 mm
- net Net-(D2-A): track 0.00 -> 5.03 mm
- net D13: track 0.00 -> 3.64 mm, vias 0 -> 1
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- added copper zone on B.Cu, net (none)
- added copper zone on B.Cu, net GND
- added copper zone on B.Cu, net S1 +
Other:
- board text added: "2A Grupo 1"
- board text added: "D18/SCK"

Commit message: PCB Terminada
Parts:
- removed ? (x3): , 
- R1, R2: footprint Resistor_THT:R_Axial_DIN0204_L3.6mm_D1.6mm_P5.08mm_Horizontal -> Resistor_THT:R_Axial_DIN0207_L6.3mm_D2.5mm_P10.16mm_Horizontal
- moved REF** 47.1 mm to (92.6, 125.4)
Connections:
- REF** pad 1: GND -> Vin
- REF** pad 2: S1 + -> (no net)
Routing:
- net Net-(D2-A): track 5.03 -> 10.2 mm
- net Net-(D1-A): track 5.58 -> 10.7 mm
- net Vin: track 29.6 -> 30.6 mm

Commit message: Ordenado
Routing:
- net GND: track 299.6 -> 201.8 mm
- net S1 +: track 297.8 -> 373.5 mm
Changed lines of the file:
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@@
 	)
 	(gr_line
-		(start 62 138)
-		(end 141 138)
+		(start 61.5 138)
+		(end 141.5 138)
 		(stroke
 			(width 0.2)
@@
 		)
 		(layer "B.Cu")
-		(net 2)
+		(net 7)
 	)
 	(gr_line
@@
 	)
 	(segment
-		(start 65.5 62)
-		(end 62.5 59)
-		(width 1)
-		(layer "B.Cu")
-		(net 2)
-	)
-	(segment
-		(start 61.5 58.5)
-		(end 61.5 138)
-		(width 0.2)
-		(layer "B.Cu")
-		(net 2)
-	)
-	(segment
 		(start 125 96.04)
 		(end 122.54 96.04)
@@
 	)
 	(segment
-		(start 69 65.5)
-		(end 65.5 62)
-		(width 1)
-		(layer "B.Cu")
-		(net 2)
-	)
-	(segment
 		(start 83.5 60)
 		(end 82.5 61)
@@
 		(start 109.1931 110.1931)
 		(end 114.944 110.1931)
-		(width 1)
-		(layer "B.Cu")
-		(net 2)
-	)
-	(segment
-		(start 65.5 62)
-		(end 68.5 59)
 		(width 1)
 		(layer "B.Cu")
@@
 		(start 122.5 96)
 		(end 120.5 98)
-		(width 1)
-		(layer "B.Cu")
-		(net 2)
-	)
-	(segment
-		(start 65.5 62)
-		(end 62 65.5)
 		(width 1)
 		(layer "B.Cu")
@@
 	)
 	(segment
+		(start 65.5 62)
+		(end 62.5 59)
+		(width 1)
+		(layer "B.Cu")
+		(net 7)
+	)
+	(segment
 		(start 114.944 112.7331)
 		(end 118.4831 112.7331)
@@
 	)
 	(segment
+		(start 61.5 58.5)
+		(end 61.5 138)
+		(width 0.2)
+		(layer "B.Cu")
+		(net 7)
+	)
+	(segment
+		(start 69 65.5)
+		(end 65.5 62)
+		(width 1)
+		(layer "B.Cu")
+		(net 7)
+	)
+	(segment
 		(start 137 134)
 		(end 134 137)
@@
 	)
 	(segment
-		(start 66 134)
-		(end 62.5 130.5)
-		(width 1)
-		(layer "B.Cu")
-		(net 7)
-	)
-	(segment
 		(start 114.944 112.7331)
 		(end 114.944 136.056)
@@
 	)
 	(segment
+		(start 65.5 62)
+		(end 68.5 59)
+		(width 1)
+		(layer "B.Cu")
+		(net 7)
+	)
+	(segment
 		(start 76 126.5)
 		(end 76 90)
@@
 	)
 	(segment
-		(start 66 134)
-		(end 68.5 136.5)
-		(width 1)
-		(layer "B.Cu")
-		(net 7)
-	)
-	(segment
 		(start 125 93.5)
 		(end 122.5 93.5)
@@
 	)
 	(segment
-		(start 66 134)
-		(end 69.5 130.5)
+		(start 65.5 62)
+		(end 62 65.5)
 		(width 1)
 		(layer "B.Cu")
@@
 		(start 78 88)
 		(end 79.5 88)
-		(width 1)
-		(layer "B.Cu")
-		(net 7)
-	)
-	(segment
-		(start 66 134)
-		(end 69 137)
 		(width 1)
 		(layer "B.Cu")
@@
 		(width 1)
 		(layer "B.Cu")
-		(net 7)
-	)
-	(segment
-		(start 66 134)
-		(end 62.801 137.199)
-		(width 1)
-		(layer "B.Cu")
